File: thermal-pcb/thermal-pcb.kicad_sch (KiCad schematic)
At the start: 11 parts, among them J1 MLX90640_Breakout, J2 Conn_01x14_Pin, J3 USB_C_Receptacle_USB2.0_16P, J4 Conn_01x04_Socket, Q1 FS8205A, U1 ESP32-S3-WROOM-1, U2 MCP73871, U3 MIC5504-3.3YM5, U4 DW01A

Commit message: work on pcb
Parts:
- added C1, C2: 4.7uF, symbol Device:C
- added C3: 10uF, symbol Device:C
- added D1: LED, symbol Device:LED
- added JP1: EN_VIN, symbol Jumper:Jumper_2_Bridged
- added JP2: EN_GND, Jumper:SolderJumper-2_P1.3mm_Open_RoundedPad1.0x1.5mm, symbol Jumper:SolderJumper_2_Open
- added R3, R4: 470, symbol Device:R
- added R5: 10k, symbol Device:R
- added TH1: 10k, symbol Device:Thermistor_NTC
- R1, R2: value R -> 5.1k
Connections:
- net GND: now also C1.2, C2.2, C3.2, JP2.1 (A), TH1.1
- net VBUS: now also U2.17 (CE), U2.18 (IN), U2.19 (IN), U2.2 (VPCC), U2.3 (SEL), U2.9 (~{TE}), C3.1
- net VCC: now also R3.2, R5.2
- net at U3.1 (VIN): now also U2.1 (OUT), U2.20 (OUT), C2.1, JP1.1 (A)
- net at U3.3 (EN): now also JP1.2 (B), JP2.2 (B)
- net +BATT: now reaches U2.14 (V_{BAT}), U2.15 (V_{BAT})
- net +BATT: now also C1.1
- net at U2.5 (THERM): now also TH1.2
- net PG: now reaches U2.6 (~{PG})
- net PG: now also D1.1 (K), R5.1
- new net: D1.2 (A), R3.1
Other:
- moved on the sheet: Q1, U2, U3

Commit message: stuff
Parts:
- added C4, C5: 1uF, Capacitor_SMD:C_0805_2012Metric, symbol Device:C
- added C6: 0.1uF, Capacitor_SMD:C_0805_2012Metric, symbol Device:C
- added D2: LED_R, LED_SMD:LED_0603_1608Metric, symbol Device:LED
- added D3: LED_G, LED_SMD:LED_0603_1608Metric, symbol Device:LED
- added J5: BATT_CONN, symbol Connector:Conn_01x02_Pin
- added R10: 4.02k, symbol Device:R
- added R11: 20k, symbol Device:R
- added R12, R13, R6, R7: 10k, symbol Device:R
- added R14: 1k, symbol Device:R
- added R8, R9: 470, symbol Device:R
- added TP1: TP_BATT+, symbol Connector:TestPoint
- added TP2: TP_VCC, symbol Connector:TestPoint
- added TP3: VBUS_TP, TestPoint:TestPoint_Pad_D2.0mm, symbol Connector:TestPoint
- added TP4: VIN_TP, TestPoint:TestPoint_Pad_D2.0mm, symbol Connector:TestPoint
- added TP5: PG_TP, TestPoint:TestPoint_Pad_D2.0mm, symbol Connector:TestPoint
- added TP6: STAT2_TP, TestPoint:TestPoint_Pad_D2.0mm, symbol Connector:TestPoint
- added TP7: STAT1_TP, TestPoint:TestPoint_Pad_D2.0mm, symbol Connector:TestPoint
- added TP8: PROT_CS, symbol Connector:TestPoint
- C1, C2, C3: footprint (none) -> Capacitor_SMD:C_0805_2012Metric
- D1: value LED -> LED_B; footprint (none) -> LED_SMD:LED_0603_1608Metric
- J1: footprint (none) -> Connector_PinSocket_2.54mm:PinSocket_1x05_P2.54mm_Vertical
- JP1: footprint (none) -> Jumper:SolderJumper-2_P1.3mm_Bridged_RoundedPad1.0x1.5mm
- R4: value 470 -> 100
Connections:
- net +BATT: now also R4.1, U2.16 (V_{BAT_SENSE}), J5.1 (Pin_1), TP1.1
- net GND: now also U2.10 (V_{SS}), U2.11 (V_{SS}), U2.21 (V_{SS}), C4.2, C5.1, J5.2 (Pin_2), R10.1, R11.2
- net I2C_SCL: now also R13.2
- net I2C_SDA: now also R12.2
- net PG: now also U1.32 (IO39), TP5.1
- net VBUS: now also U2.4 (PROG2), TP3.1
- net VCC: now also U3.5 (VOUT), C4.1, R12.1, R13.1, R6.2, R7.2, R8.2, R9.2, TP2.1
- net at C2.1, JP1.1 (A), U2.1 (OUT)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: now also C5.2, TP4.1
- net at R4.2: now also U4.5 (VCC), C6.1
- net STAT2: now reaches U1.33 (IO40)
- net STAT2: now also U2.7 (STAT2), D2.1 (K), R6.1, TP6.1
- net STAT1: now reaches U1.34 (IO41)
- net STAT1: now also U2.8 (STAT1/~{LBO}), D3.1 (K), R7.1, TP7.1
- net at U4.1 (OD): now also Q1.4
- net at U4.2 (CS): now also R14.2, TP8.1
- net at U4.3 (OC): now also Q1.5
- net at U4.6 (GND): now also Q1.2, Q1.3, C6.2
- net at U2.12 (PROG3): now also R11.1
- net at U2.13 (PROG1): now also R10.2
- net at Q1.6, Q1.7: now also R14.1
- new net: D2.2 (A), R8.1
- new net: D3.2 (A), R9.1
Other:
- moved on the sheet: C1, D1, Q1, R3, R5, TH1, U4

Commit message: work on schematic
Parts:
- J2: footprint (none) -> Connector_PinSocket_2.54mm:PinSocket_1x14_P2.54mm_Vertical
- J3: footprint (none) -> Connector_USB:USB_C_Receptacle_G-Switch_GT-USB-7010ASV
- J4: footprint (none) -> Connector_PinSocket_2.54mm:PinSocket_1x04_P2.54mm_Vertical
- J5: footprint (none) -> Connector_PinSocket_2.54mm:PinSocket_1x02_P2.54mm_Vertical
- Q1: footprint FS8205A:SOP65P640X120-8N -> Component:SOP65P640X120-8N
- R1, R10, R11, R12, R13, R14, R2, R3, R4, R5, R6, R7, R8, R9, TH1: footprint (none) -> Resistor_SMD:R_0805_2012Metric
- TP1, TP2, TP8: footprint (none) -> TestPoint:TestPoint_Pad_D2.0mm
Changed lines of the file:
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@@
 			)
 		)
-		(property "Footprint" ""
+		(property "Footprint" "Resistor_SMD:R_0805_2012Metric"
 			(at 270.51 152.908 90)
 			(effects
@@
 			)
 		)
-		(property "Footprint" ""
+		(property "Footprint" "Connector_PinSocket_2.54mm:PinSocket_1x14_P2.54mm_Vertical"
 			(at 33.02 57.15 0)
 			(effects
@@
 			)
 		)
-		(property "Footprint" ""
+		(property "Footprint" "Resistor_SMD:R_0805_2012Metric"
 			(at 184.15 74.168 90)
 			(effects
@@
 			)
 		)
-		(property "Footprint" ""
+		(property "Footprint" "Resistor_SMD:R_0805_2012Metric"
 			(at 73.66 104.648 90)
 			(effects
@@
 			)
 		)
-		(property "Footprint" ""
+		(property "Footprint" "Resistor_SMD:R_0805_2012Metric"
 			(at 130.81 51.308 90)
 			(effects
@@
 			)
 		)
-		(property "Footprint" ""
+		(property "Footprint" "Resistor_SMD:R_0805_2012Metric"
 			(at 203.2 70.358 90)
 			(effects
@@
 			)
 		)
-		(property "Footprint" ""
+		(property "Footprint" "Resistor_SMD:R_0805_2012Metric"
 			(at 270.51 161.798 90)
 			(effects
@@
 			)
 		)
-		(property "Footprint" ""
+		(property "Footprint" "Resistor_SMD:R_0805_2012Metric"
 			(at 272.288 113.03 90)
 			(effects
@@
 			)
 		)
-		(property "Footprint" ""
+		(property "Footprint" "TestPoint:TestPoint_Pad_D2.0mm"
 			(at 271.78 104.14 0)
 			(effects
@@
 			)
 		)
-		(property "Footprint" ""
+		(property "Footprint" "Resistor_SMD:R_0805_2012Metric"
 			(at 223.52 98.298 90)
 			(effects
@@
 			)
 		)
-		(property "Footprint" ""
+		(property "Footprint" "TestPoint:TestPoint_Pad_D2.0mm"
 			(at 265.43 44.45 0)
 			(effects
@@
 			)
 		)
-		(property "Footprint" ""
+		(property "Footprint" "Resistor_SMD:R_0805_2012Metric"
 			(at 138.43 52.832 90)
 			(effects
@@
 			)
 		)
-		(property "Footprint" ""
+		(property "Footprint" "Connector_USB:USB_C_Receptacle_G-Switch_GT-USB-7010ASV"
 			(at 46.99 110.49 0)
 			(effects
@@
 			)
 		)
-		(property "Footprint" ""
+		(property "Footprint" "Resistor_SMD:R_0805_2012Metric"
 			(at 76.962 130.81 90)
 			(effects
@@
 			)
 		)
-		(property "Footprint" ""
+		(property "Footprint" "Connector_PinSocket_2.54mm:PinSocket_1x02_P2.54mm_Vertical"
 			(at 245.11 78.74 0)
 			(effects
@@
 			)
 		)
-		(property "Footprint" ""
+		(property "Footprint" "Resistor_SMD:R_0805_2012Metric"
 			(at 73.66 98.552 90)
 			(effects
@@
 			)
 		)
-		(property "Footprint" ""
+		(property "Footprint" "TestPoint:TestPoint_Pad_D2.0mm"
 			(at 270.51 76.2 0)
 			(effects
@@
 			)
 		)
-		(property "Footprint" ""
+		(property "Footprint" "Connector_PinSocket_2.54mm:PinSocket_1x04_P2.54mm_Vertical"
 			(at 80.01 57.15 0)
 			(effects
@@
 			)
 		)
-		(property "Footprint" ""
+		(property "Footprint" "Resistor_SMD:R_0805_2012Metric"
 			(at 129.54 69.85 0)
 			(effects
@@
 			)
 		)
-		(property "Footprint" ""
+		(property "Footprint" "Resistor_SMD:R_0805_2012Metric"
 			(at 68.072 130.81 90)
 			(effects
@@
 			)
 		)
-		(property "Footprint" "FS8205A:SOP65P640X120-8N"
+		(property "Footprint" "Component:SOP65P640X120-8N"
 			(at 252.73 121.92 0)
 			(effects
@@
 			)
 		)
-		(property "Footprint" ""
+		(property "Footprint" "Resistor_SMD:R_0805_2012Metric"
 			(at 270.51 144.018 90)
 			(effects
@@
 			)
 		)
-		(property "Footprint" ""
+		(property "Footprint" "Resistor_SMD:R_0805_2012Metric"
 			(at 185.42 66.548 90)
 			(effects

Commit message: schematic
Connections:
- net GND: now also Q1.6, Q1.7, R14.1; no longer J5.2 (Pin_2)
- net -BATT: now reaches C6.2, Q1.2, Q1.3, U4.6 (GND)
- net -BATT: now also J5.2 (Pin_2)
Changed lines of the file:
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@@
 	(paper "A4")
 	(junction
+		(at 270.51 121.92)
+		(diameter 0)
+		(color 0 0 0 0)
+	)
+	(junction
 		(at 220.98 39.37)
 		(diameter 0)
@@
 	)
 	(junction
+		(at 228.6 121.92)
+		(diameter 0)
+		(color 0 0 0 0)
+	)
+	(junction
 		(at 177.8 52.07)
 		(diameter 0)
@@
 	(wire
 		(pts
-			(xy 228.6 121.92) (xy 228.6 104.14)
+			(xy 228.6 104.14) (xy 228.6 121.92)
 		)
 		(stroke
@@
 	)
 	(symbol
+		(lib_id "power:-BATT")
+		(at 228.6 121.92 90)
+		(unit 1)
+		(exclude_from_sim no)
+		(in_bom yes)
+		(on_board yes)
+		(dnp no)
+		(fields_autoplaced yes)
+		(property "Reference" "#PWR042"
+			(at 232.41 121.92 0)
+			(effects
+				(font
+					(size 1.27 1.27)
+				)
+				(hide yes)
+			)
+		)
+		(property "Value" "-BATT"
+			(at 224.79 121.9199 90)
+			(effects
+				(font
+					(size 1.27 1.27)
+				)
+				(justify left)
+			)
+		)
+		(property "Footprint" ""
+			(at 228.6 121.92 0)
+			(effects
+				(font
+					(size 1.27 1.27)
+				)
+				(hide yes)
+			)
+		)
+		(property "Datasheet" ""
+			(at 228.6 121.92 0)
+			(effects
+				(font
+					(size 1.27 1.27)
+				)
+				(hide yes)
+			)
+		)
+		(property "Description" "Power symbol creates a global label with name \"-BATT\""
+			(at 228.6 121.92 0)
+			(effects
+				(font
+					(size 1.27 1.27)
+				)
+				(hide yes)
+			)
+		)
+		(pin "1"
+		)
+		(instances
+			(project "thermal-pcb"
+				(path "/e071f646-3958-4d62-9e1f-6199960ec462"
+					(reference "#PWR042")
+					(unit 1)
+				)
+			)
+		)
+	)
+	(symbol
 		(lib_id "power:GND")
 		(at 242.57 49.53 0)
@@
 	)
 	(symbol
-		(lib_id "power:GND")
-		(at 250.19 81.28 90)
-		(mirror x)
-		(unit 1)
-		(exclude_from_sim no)
-		(in_bom yes)
-		(on_board yes)
-		(dnp no)
-		(fields_autoplaced yes)
-		(property "Reference" "#PWR014"
-			(at 256.54 81.28 0)
-			(effects
-				(font
-					(size 1.27 1.27)
-				)
-				(hide yes)
-			)
-		)
-		(property "Value" "GND"
-			(at 254 81.2799 90)
-			(effects
-				(font
-					(size 1.27 1.27)
-				)
-				(justify right)
-			)
-		)
-		(property "Footprint" ""
-			(at 250.19 81.28 0)
-			(effects
-				(font
-					(size 1.27 1.27)
-				)
-				(hide yes)
-			)
-		)
-		(property "Datasheet" ""
-			(at 250.19 81.28 0)
-			(effects
-				(font
-					(size 1.27 1.27)
-				)
-				(hide yes)
-			)
-		)
-		(property "Description" "Power symbol creates a global label with name \"GND\" , ground"
-			(at 250.19 81.28 0)
-			(effects
-				(font
-					(size 1.27 1.27)
-				)
-				(hide yes)
-			)
-		)
-		(pin "1"
-		)
-		(instances
-			(project "thermal-pcb"
-				(path "/e071f646-3958-4d62-9e1f-6199960ec462"
-					(reference "#PWR014")
-					(unit 1)
-				)
-			)
-		)
-	)
-	(symbol
 		(lib_id "power:VCC")
 		(at 189.23 64.77 270)
@@
 	)
 	(symbol
+		(lib_id "power:GND")
+		(at 270.51 121.92 90)
+		(mirror x)
+		(unit 1)
+		(exclude_from_sim no)
+		(in_bom yes)
+		(on_board yes)
+		(dnp no)
+		(property "Reference" "#PWR043"
+			(at 276.86 121.92 0)
+			(effects
+				(font
+					(size 1.27 1.27)
+				)
+				(hide yes)
+			)
+		)
+		(property "Value" "GND"
+			(at 275.59 121.92 0)
+			(effects
+				(font
+					(size 1.27 1.27)
+				)
+			)
+		)
+		(property "Footprint" ""
+			(at 270.51 121.92 0)
+			(effects
+				(font
+					(size 1.27 1.27)
+				)
+				(hide yes)
+			)
+		)
+		(property "Datasheet" ""
+			(at 270.51 121.92 0)
+			(effects
+				(font
+					(size 1.27 1.27)
+				)
+				(hide yes)
+			)
+		)
+		(property "Description" "Power symbol creates a global label with name \"GND\" , ground"
+			(at 270.51 121.92 0)
+			(effects
+				(font
+					(size 1.27 1.27)
+				)
+				(hide yes)
+			)
+		)
+		(pin "1"
+		)
+		(instances
+			(project "thermal-pcb"
+				(path "/e071f646-3958-4d62-9e1f-6199960ec462"
+					(reference "#PWR043")
+					(unit 1)
+				)
+			)
+		)
+	)
+	(symbol
 		(lib_id "power:VCC")
 		(at 115.57 96.52 0)
@@
 					(unit 1)
 				)
+			)
+		)
+	)
+	(symbol
+		(lib_id "power:-BATT")
+		(at 250.19 81.28 270)
+		(unit 1)
+		(exclude_from_sim no)
+		(in_bom yes)
+		(on_board yes)
+		(dnp no)
+		(fields_autoplaced yes)
+		(property "Reference" "#PWR020"
+			(at 246.38 81.28 0)
+			(effects
+				(font
+					(size 1.27 1.27)
+				)
+				(hide yes)
+			)
+		)
+		(property "Value" "-BATT"
+			(at 254 81.2799 90)
+			(effects
+				(font
+					(size 1.27 1.27)
+				)
+				(justify left)
+			)
+		)
+		(property "Footprint" ""
+			(at 250.19 81.28 0)
+			(effects
+				(font
+					(size 1.27 1.27)
+				)
+				(hide yes)
+			)
+		)
+		(property "Datasheet" ""
+			(at 250.19 81.28 0)
+			(effects
+				(font
+					(size 1.27 1.27)
+				)
+				(hide yes)
+			)
+		)
+		(property "Description" "Power symbol creates a global label with name \"-BATT\""
+			(at 250.19 81.28 0)
+			(effects
+				(font
+					(size 1.27 1.27)
+				)
+				(hide yes)
+			)
+		)
+		(pin "1"
+		)
+		(instances
+			(project ""
+				(path "/e071f646-3958-4d62-9e1f-6199960ec462"
+					(reference "#PWR020")
+					(unit 1)
+				)

Commit message: 5/31
Parts:
- added JP3: PROG1_JP, Jumper:SolderJumper-2_P1.3mm_Bridged_RoundedPad1.0x1.5mm, symbol Jumper:SolderJumper_2_Bridged
- added JP4: PROG2_JP, Jumper:SolderJumper-2_P1.3mm_Bridged_RoundedPad1.0x1.5mm, symbol Jumper:SolderJumper_2_Bridged
- added JP5: PROG3_JP, Jumper:SolderJumper-2_P1.3mm_Bridged_RoundedPad1.0x1.5mm, symbol Jumper:SolderJumper_2_Bridged
- added JP6: SEL_JP, Jumper:SolderJumper-2_P1.3mm_Bridged_RoundedPad1.0x1.5mm, symbol Jumper:SolderJumper_2_Bridged
- added JP7: PG_JP, Jumper:SolderJumper-2_P1.3mm_Bridged_RoundedPad1.0x1.5mm, symbol Jumper:SolderJumper_2_Bridged
- added JP8: STAT1_JP, Jumper:SolderJumper-2_P1.3mm_Bridged_RoundedPad1.0x1.5mm, symbol Jumper:SolderJumper_2_Bridged
- added JP9: STAT2_JP, Jumper:SolderJumper-2_P1.3mm_Bridged_RoundedPad1.0x1.5mm, symbol Jumper:SolderJumper_2_Bridged
- added TP10: SDA_TP, TestPoint:TestPoint_Pad_D1.5mm, symbol Connector:TestPoint
- added TP11: SCL_TP, TestPoint:TestPoint_Pad_D1.5mm, symbol Connector:TestPoint
- added TP9: MOSFET_P8, TestPoint:TestPoint_Pad_D1.5mm, symbol Connector:TestPoint
- TP1, TP2, TP3, TP4, TP5, TP6, TP7, TP8: footprint TestPoint:TestPoint_Pad_D2.0mm -> TestPoint:TestPoint_Pad_D1.5mm
Connections:
- net I2C_SCL: now also TP11.1
- net I2C_SDA: now also TP10.1
- net PG: now also JP7.2 (B); no longer U2.6 (~{PG})
- net STAT1: now also JP8.2 (B); no longer U2.8 (STAT1/~{LBO})
- net STAT2: now also JP9.2 (B); no longer U2.7 (STAT2)
- net VBUS: now also JP4.2 (B), JP6.2 (B); no longer U2.3 (SEL), U2.4 (PROG2)
- net at R10.2: now also JP3.1 (A); no longer U2.13 (PROG1)
- net at U2.12 (PROG3): now also JP5.1 (A); no longer R11.1
- net at Q1.1, Q1.8: now also TP9.1
- new net: JP9.1 (A), U2.7 (STAT2)
- new net: JP5.2 (B), R11.1
- new net: JP4.1 (A), U2.4 (PROG2)
- new net: JP8.1 (A), U2.8 (STAT1/~{LBO})
- new net: JP3.2 (B), U2.13 (PROG1)
- new net: JP6.1 (A), U2.3 (SEL)
- new net: JP7.1 (A), U2.6 (~{PG})
Other:
- moved on the sheet: C1, C2, C3, C4, C5, J5, JP1, JP2, R10, R11, R12, R13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

Commit message: work
Parts:
- removed JP1: EN_VIN, Jumper:SolderJumper-2_P1.3mm_Bridged_RoundedPad1.0x1.5mm, symbol Jumper:Jumper_2_Bridged
- added C7: 22uF, Capacitor_SMD:C_0805_2012Metric, symbol Device:C
- added F1: 1.5A, Fuse:Fuse_1206_3216Metric, symbol Device:Fuse
- added JP1: EN_VCC, Jumper:SolderJumper-2_P1.3mm_Bridged_RoundedPad1.0x1.5mm, symbol Jumper:SolderJumper_2_Bridged
- added Q2: AO3415, AO3415:SOT-23-3_L2.9-W1.3-P1.90-LS2.4-BR, symbol AO3415:AO3415_C181094
Connections:
- net GND is gone; now on net -BATT: C1.2, C2.2, C3.2, C4.2, C5.1, J1.3 (Pin_3), J2.2 (Pin_2), J3.A1 (GND), J3.A12 (GND), J3.B1 (GND), J3.B12 (GND), J3.S1 (SHIELD), J4.1 (Pin_1), JP2.1 (A), Q1.6, Q1.7, R1.2, R10.1, R11.2, R14.1, R2.1, TH1.1, U1.1 (GND), U1.40 (GND), U1.41 (GND), U2.10 (V_{SS}), U2.11 (V_{SS}), U2.21 (V_{SS}), U3.2 (GND)
- net +BATT: now also C7.1, Q2.2 (S); no longer J5.1 (Pin_1)
- net -BATT: now also C7.2, Q2.1 (G)
- net VBUS: now also F1.2; no longer J3.A4 (VBUS), J3.A9 (VBUS), J3.B4 (VBUS), J3.B9 (VBUS)
- net at C2.1, C5.2, TP4.1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: now also JP1.1 (A)
- net at JP2.2 (B), U3.3 (EN): now also JP1.2 (B)
- new net: F1.1, J3.A4 (VBUS), J3.A9 (VBUS), J3.B4 (VBUS), J3.B9 (VBUS)
- new net: J5.1 (Pin_1), Q2.3 (D)
Other:
- moved on the sheet: J1, J2, J4, J5

Commit message: route most traces
Parts:
- Q2: footprint AO3415:SOT-23-3_L2.9-W1.3-P1.90-LS2.4-BR -> Component:SOT-23-3_L2.9-W1.3-P1.90-LS2.4-BR
Changed lines of the file:
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@@
 			)
 		)
-		(property "Footprint" "AO3415:SOT-23-3_L2.9-W1.3-P1.90-LS2.4-BR"
+		(property "Footprint" "Component:SOT-23-3_L2.9-W1.3-P1.90-LS2.4-BR"
 			(at 167.64 109.22 0)
 			(effects
