File: thermal-pcb/thermal-pcb.kicad_sch (KiCad schematic)
At the start: 57 parts, among them J1 MLX90640_Breakout, J2 Conn_01x14_Pin, J3 USB_C_Receptacle_USB2.0_16P, J4 Conn_01x04_Socket, J5 BATT_CONN, Q1 FS8205A, Q2 AO3415, U1 ESP32-S3-WROOM-1, U2 MCP73871, U3 MIC5504-3.3YM5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

Commit message: some stuff
Parts:
- removed J1: MLX90640_Breakout, Connector_PinSocket_2.54mm:PinSocket_1x05_P2.54mm_Vertical, symbol Connector:Conn_01x05_Socket
- added C8: 1uF, Capacitor_SMD:C_0805_2012Metric, symbol Device:C
- added C9: 0.1uF, Capacitor_SMD:C_0805_2012Metric, symbol Device:C
- added JP10: VCC_JP, Jumper:SolderJumper-2_P1.3mm_Bridged_RoundedPad1.0x1.5mm, symbol Jumper:SolderJumper_2_Bridged
- added U5: MLX90640ESF-BAB-000-SP, Component:TO292P945H1165-4, symbol MLX90640ESF-BAB-000-SP:MLX90640ESF-BAB-000-SP
- R12, R13: value 10k -> 2.2k
Connections:
- net -BATT: now also C8.2, C9.2, U5.3 (GND)
- net I2C_SCL: now also U5.4 (SCL)
- net I2C_SDA: now also U5.1 (SDA)
- net VCC: now also C8.1, C9.1, JP10.1 (A), U5.2 (VDD); no longer C4.1, TP2.1, U3.5 (VOUT)
- new net: C4.1, JP10.2 (B), TP2.1, U3.5 (VOUT)

Commit message: work on pcb
Parts:
- J3: footprint Connector_USB:USB_C_Receptacle_G-Switch_GT-USB-7010ASV -> Connector_USB:USB_C_Receptacle_GCT_USB4105-xx-A_16P_TopMnt_Horizontal
Changed lines of the file:
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@@
 			)
 		)
-		(property "Footprint" "Connector_USB:USB_C_Receptacle_G-Switch_GT-USB-7010ASV"
+		(property "Footprint" "Connector_USB:USB_C_Receptacle_GCT_USB4105-xx-A_16P_TopMnt_Horizontal"
 			(at 46.99 110.49 0)
 			(effects

Commit message: 6/3
Parts:
- added J1: FALLBACK_IN, Connector_PinHeader_2.54mm:PinHeader_1x02_P2.54mm_Vertical, symbol Connector:Conn_01x02_Pin
- added JP11: BMS_VOUT, Jumper:SolderJumper-2_P1.3mm_Bridged_RoundedPad1.0x1.5mm, symbol Jumper:SolderJumper_2_Bridged
Connections:
- net -BATT: now also J1.2 (Pin_2)
- net at C2.1, TP4.1, U2.1 (OUT)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: now also JP11.2 (B); no longer C5.2, JP1.1 (A), U3.1 (VIN)
- new net: C5.2, J1.1 (Pin_1), JP1.1 (A), JP11.1 (A), U3.1 (VIN)
Other:
- moved on the sheet: C2, TP4

Commit message: almost done pcb
Parts:
- added JP12: FUSE_BYPASS, Jumper:SolderJumper-2_P1.3mm_Open_RoundedPad1.0x1.5mm, symbol Jumper:SolderJumper_2_Open
Connections:
- net VBUS: now also JP12.2 (B)
- net at F1.1, J3.A4 (VBUS), J3.A9 (VBUS)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: now also JP12.1 (A)
Changed lines of the file:
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@@
 	)
 	(junction
+		(at 73.66 95.25)
+		(diameter 0)
+		(color 0 0 0 0)
+	)
+	(junction
 		(at 128.27 21.59)
 		(diameter 0)
@@
 	(wire
 		(pts
+			(xy 73.66 95.25) (xy 58.42 95.25)
+		)
+		(stroke
+			(width 0)
+			(type default)
+		)
+	)
+	(wire
+		(pts
 			(xy 226.06 45.72) (xy 226.06 46.99)
 		)
@@
 	(wire
 		(pts
+			(xy 73.66 91.44) (xy 73.66 95.25)
+		)
+		(stroke
+			(width 0)
+			(type default)
+		)
+	)
+	(wire
+		(pts
 			(xy 144.78 69.85) (xy 147.32 69.85)
 		)
@@
 	(wire
 		(pts
-			(xy 78.74 95.25) (xy 58.42 95.25)
+			(xy 78.74 95.25) (xy 73.66 95.25)
 		)
 		(stroke
@@
 		(on_board yes)
 		(dnp no)
-		(fields_autoplaced yes)
 		(property "Reference" "F1"
-			(at 82.55 88.9 90)
+			(at 82.55 90.424 90)
 			(effects
 				(font
@@
 		)
 		(property "Value" "1.5A"
-			(at 82.55 91.44 90)
+			(at 82.55 92.964 90)
 			(effects
 				(font
@@
 	)
 	(symbol
+		(lib_id "Jumper:SolderJumper_2_Open")
+		(at 73.66 87.63 90)
+		(unit 1)
+		(exclude_from_sim no)
+		(in_bom no)
+		(on_board yes)
+		(dnp no)
+		(fields_autoplaced yes)
+		(property "Reference" "JP12"
+			(at 76.2 86.3599 90)
+			(effects
+				(font
+					(size 1.27 1.27)
+				)
+				(justify right)
+				(hide yes)
+			)
+		)
+		(property "Value" "FUSE_BYPASS"
+			(at 76.2 88.8999 90)
+			(effects
+				(font
+					(size 1.27 1.27)
+				)
+				(justify right)
+				(hide yes)
+			)
+		)
+		(property "Footprint" "Jumper:SolderJumper-2_P1.3mm_Open_RoundedPad1.0x1.5mm"
+			(at 73.66 87.63 0)
+			(effects
+				(font
+					(size 1.27 1.27)
+				)
+				(hide yes)
+			)
+		)
+		(property "Datasheet" "~"
+			(at 73.66 87.63 0)
+			(effects
+				(font
+					(size 1.27 1.27)
+				)
+				(hide yes)
+			)
+		)
+		(property "Description" "Solder Jumper, 2-pole, open"
+			(at 73.66 87.63 0)
+			(effects
+				(font
+					(size 1.27 1.27)
+				)
+				(hide yes)
+			)
+		)
+		(pin "2"
+		)
+		(pin "1"
+		)
+		(instances
+			(project "thermal-pcb"
+				(path "/e071f646-3958-4d62-9e1f-6199960ec462"
+					(reference "JP12")
+					(unit 1)
+				)
+			)
+		)
+	)
+	(symbol
 		(lib_id "Battery_Management:DW01A")
 		(at 250.19 101.6 0)
@@
 					(unit 1)
 				)
+			)
+		)
+	)
+	(symbol
+		(lib_id "power:VBUS")
+		(at 73.66 83.82 270)
+		(unit 1)
+		(exclude_from_sim no)
+		(in_bom yes)
+		(on_board yes)
+		(dnp no)
+		(fields_autoplaced yes)
+		(property "Reference" "#PWR049"
+			(at 69.85 83.82 0)
+			(effects
+				(font
+					(size 1.27 1.27)
+				)
+				(hide yes)
+			)
+		)
+		(property "Value" "VBUS"
+			(at 77.47 83.8199 90)
+			(effects
+				(font
+					(size 1.27 1.27)
+				)
+				(justify left)
+			)
+		)
+		(property "Footprint" ""
+			(at 73.66 83.82 0)
+			(effects
+				(font
+					(size 1.27 1.27)
+				)
+				(hide yes)
+			)
+		)
+		(property "Datasheet" ""
+			(at 73.66 83.82 0)
+			(effects
+				(font
+					(size 1.27 1.27)
+				)
+				(hide yes)
+			)
+		)
+		(property "Description" "Power symbol creates a global label with name \"VBUS\""
+			(at 73.66 83.82 0)
+			(effects
+				(font
+					(size 1.27 1.27)
+				)
+				(hide yes)
+			)
+		)
+		(pin "1"
+		)
+		(instances
+			(project "thermal-pcb"
+				(path "/e071f646-3958-4d62-9e1f-6199960ec462"
+					(reference "#PWR049")
+					(unit 1)
+				)

Commit message: finish pcb
Parts:
- D1, D2, D3: footprint LED_SMD:LED_0603_1608Metric -> LED_SMD:LED_1206_3216Metric
Changed lines of the file:
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@@
 			)
 		)
-		(property "Footprint" "LED_SMD:LED_0603_1608Metric"
+		(property "Footprint" "LED_SMD:LED_1206_3216Metric"
 			(at 262.89 142.24 0)
 			(effects
@@
 			)
 		)
-		(property "Footprint" "LED_SMD:LED_0603_1608Metric"
+		(property "Footprint" "LED_SMD:LED_1206_3216Metric"
 			(at 262.89 160.02 0)
 			(effects
@@
 			)
 		)
-		(property "Footprint" "LED_SMD:LED_0603_1608Metric"
+		(property "Footprint" "LED_SMD:LED_1206_3216Metric"
 			(at 262.89 151.13 0)
 			(effects

Commit message: add firmware
Parts:
- removed Q1: FS8205A, Component:SOP65P640X120-8N, symbol FS8205A:FS8205A
- added H1, H2, H3, H4: MountingHole, MountingHole:MountingHole_4.3mm_M4, symbol Mechanical:MountingHole
- added Q1: FS8205, Component:SOT95P280X145-6N, symbol FS8205:FS8205
- added SW1: MFS201N-16-Z, Component:MFS201N-16-Z_NDC, symbol switch:MFS201N-16-Z
Connections:
- net -BATT: now also Q1.1, Q1.3
- net at TP9.1: now also Q1.2, Q1.5
- net at Q2.3 (D): now also SW1.4; no longer J5.1 (Pin_1)
- net at U4.1 (OD): now also Q1.6
- net at U4.3 (OC): now also Q1.4
- new net: J5.1 (Pin_1), SW1.5
- no-connect marks 2 -> 9
Other:
- moved on the sheet: C7, J5, Q2
