File: thermal-pcb/thermal-pcb.kicad_pcb (KiCad board)
At the start: 2 copper layers, 52.5 x 50 mm, 44 parts, among them J1 MLX90640_Breakout, J2 Conn_01x14_Pin, J3 USB_C_Receptacle_USB2.0_16P, J4 Conn_01x04_Socket, J5 BATT_CONN, Q1 FS8205A, U1 ESP32-S3-WROOM-1, U2 MCP73871, U3 MIC5504-3.3YM5, U4 DW01A

Commit message: 5/31
Parts:
- added JP3: PROG1_JP, Jumper:SolderJumper-2_P1.3mm_Bridged_RoundedPad1.0x1.5mm, B.Cu at (90.0, 174.2)
- added JP4: PROG2_JP, Jumper:SolderJumper-2_P1.3mm_Bridged_RoundedPad1.0x1.5mm, B.Cu at (69.4, 169.0)
- added JP5: PROG3_JP, Jumper:SolderJumper-2_P1.3mm_Bridged_RoundedPad1.0x1.5mm, B.Cu at (90.7, 162.2)
- added JP6: SEL_JP, Jumper:SolderJumper-2_P1.3mm_Bridged_RoundedPad1.0x1.5mm, B.Cu at (69.3, 171.8)
- added JP7: PG_JP, Jumper:SolderJumper-2_P1.3mm_Bridged_RoundedPad1.0x1.5mm, B.Cu at (64.6, 162.2)
- added JP8: STAT1_JP, Jumper:SolderJumper-2_P1.3mm_Bridged_RoundedPad1.0x1.5mm, B.Cu at (78.0, 159.0)
- added JP9: STAT2_JP, Jumper:SolderJumper-2_P1.3mm_Bridged_RoundedPad1.0x1.5mm, B.Cu at (71.4, 156.0)
- added TP10: SDA_TP, TestPoint:TestPoint_Pad_D1.5mm, F.Cu at (127.0, 150.0)
- added TP11: SCL_TP, TestPoint:TestPoint_Pad_D1.5mm, F.Cu at (123.0, 166.0)
- added TP9: MOSFET_P8, TestPoint:TestPoint_Pad_D1.5mm, B.Cu at (110.8, 155.0)
- C2, C3, C4, C5, C6, D1, D2, D3, J3, Q1, R1, R10, R11, R12, R13, R14, R2, R3, R4, R5, R6, R7, R8, R9, TH1, U2, U3, U4: moved to B.Cu
- TP1, TP3, TP5, TP6: footprint TestPoint:TestPoint_Pad_D2.0mm -> TestPoint:TestPoint_Pad_D1.5mm; moved to B.Cu
- TP2, TP4, TP7, TP8: footprint TestPoint:TestPoint_Pad_D2.0mm -> TestPoint:TestPoint_Pad_D1.5mm
- moved U3 159.8 mm to (59.0, 168.0)
- moved C2 142.4 mm to (58.0, 172.0)
- moved D1 142.0 mm to (67.8, 159.2)
- moved TP4 139.6 mm to (57.0, 175.0)
- moved D2 137.2 mm to (71.5, 159.0), turned to 180 degrees
- moved C5 136.5 mm to (59.0, 175.0)
- moved C1 134.4 mm to (86.4, 170.0)
- moved JP1 132.2 mm to (60.0, 171.0)
- moved C4 131.8 mm to (64.0, 169.0)
- moved R1 131.5 mm to (64.0, 177.8), turned to 180 degrees
- moved TP5 128.5 mm to (64.5, 159.2)
- moved JP2 127.4 mm to (60.0, 168.0)
- moved C3 124.4 mm to (77.7, 163.2)
- moved U2 124.1 mm to (75.0, 170.0)
- moved TP3 122.9 mm to (74.0, 163.2)
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Connections:
- C6 pad 2: Net-(U4-GND) -> -BATT
- J5 pad 2: GND -> -BATT
- Q1 pad 2: Net-(U4-GND) -> -BATT
- Q1 pad 3: Net-(U4-GND) -> -BATT
- Q1 pad 6: Net-(Q1-Pad6) -> GND
- Q1 pad 7: Net-(Q1-Pad6) -> GND
- R10 pad 2: Net-(U2-PROG1) -> Net-(JP3-A)
- R11 pad 1: Net-(U2-PROG3) -> Net-(JP5-B)
- R14 pad 1: Net-(Q1-Pad6) -> GND
- U2 pad 12: Net-(U2-PROG3) -> Net-(JP5-A)
- U2 pad 13: Net-(U2-PROG1) -> Net-(JP3-B)
- U2 pad 3: VBUS -> Net-(JP6-A)
- U2 pad 4: VBUS -> Net-(JP4-A)
- U2 pad 6: PG -> Net-(JP7-A)
- U2 pad 7: STAT2 -> Net-(JP9-A)
- U2 pad 8: STAT1 -> Net-(JP8-A)
- U4 pad 6: Net-(U4-GND) -> -BATT
Routing:
- net VCC: track 0.00 -> 80.9 mm
- net STAT2: track 0.00 -> 62.7 mm
- net Net-(JP1-A): track 0.00 -> 34.4 mm, vias 0 -> 4
- net Net-(U4-VCC): track 0.00 -> 20.0 mm
- net Net-(JP5-A): track 0.00 -> 16.5 mm
- net -BATT: track 0.00 -> 16.3 mm
- net VBUS: track 0.00 -> 14.5 mm, vias 0 -> 2
- net Net-(JP3-B): track 0.00 -> 14.2 mm
- net Net-(JP9-A): track 0.00 -> 13.6 mm
- net Net-(JP7-A): track 0.00 -> 12.9 mm
- net Net-(JP8-A): track 0.00 -> 12.1 mm
- net Net-(J3-CC1): track 0.00 -> 9.33 mm
- net PG: track 0.00 -> 9.15 mm
- net Net-(JP1-B): track 0.00 -> 7.88 mm, vias 0 -> 1
- net Net-(J3-CC2): track 0.00 -> 7.62 mm
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- added copper zone on F.Cu, net +BATT
- added copper zone on B.Cu, net GND
- added copper zone on F.Cu, net GND
- added copper zone on B.Cu, net VBUS
Other:
- board size 52.5 x 50 mm -> 98 x 56 mm

Commit message: route most traces
Parts:
- added C7: 22uF, Capacitor_SMD:C_0805_2012Metric, B.Cu at (87.0, 166.0)
- added F1: 1.5A, Fuse:Fuse_1206_3216Metric, B.Cu at (65.0, 172.0)
- added Q2: AO3415, Component:SOT-23-3_L2.9-W1.3-P1.90-LS2.4-BR, B.Cu at (87.0, 170.0)
- JP1: value EN_VIN -> EN_VCC
Connections:
- C1 pad 2: GND -> -BATT
- C2 pad 2: GND -> -BATT
- C3 pad 2: GND -> -BATT
- C4 pad 2: GND -> -BATT
- C5 pad 1: GND -> -BATT
- J1 pad 3: GND -> -BATT
- J2 pad 2: GND -> -BATT
- J3 pad A1: GND -> -BATT
- J3 pad A12: GND -> -BATT
- J3 pad A4: VBUS -> Net-(F1-Pad1)
- J3 pad A9: VBUS -> Net-(F1-Pad1)
- J3 pad B1: GND -> -BATT
- J3 pad B12: GND -> -BATT
- J3 pad B4: VBUS -> Net-(F1-Pad1)
- J3 pad B9: VBUS -> Net-(F1-Pad1)
- J3 pad S1: GND -> -BATT
- J4 pad 1: GND -> -BATT
- J5 pad 1: +BATT -> Net-(J5-Pin_1)
- JP2 pad 1: GND -> -BATT
- Q1 pad 6: GND -> -BATT
- Q1 pad 7: GND -> -BATT
- R1 pad 2: GND -> -BATT
- R10 pad 1: GND -> -BATT
- R11 pad 2: GND -> -BATT
- R14 pad 1: GND -> -BATT
- R2 pad 1: GND -> -BATT
- TH1 pad 1: GND -> -BATT
- U1 pad 1: GND -> -BATT
- U1 pad 40: GND -> -BATT
- U1 pad 41: GND -> -BATT
- U2 pad 10: GND -> -BATT
- U2 pad 11: GND -> -BATT
- U2 pad 21: GND -> -BATT
- U3 pad 2: GND -> -BATT
Routing:
- net VCC: track 80.9 -> 214.4 mm, vias 0 -> 2
- net LCD_SDI: track 0.00 -> 100.9 mm, vias 0 -> 2
- net LCD_T_DO: track 0.00 -> 100.5 mm, vias 0 -> 2
- net LCD_DC: track 0.00 -> 97.1 mm, vias 0 -> 2
- net LCD_SCK: track 0.00 -> 95.5 mm, vias 0 -> 1
- net LCD_CS: track 0.00 -> 91.5 mm, vias 0 -> 1
- net LCD_REST: track 0.00 -> 90.1 mm, vias 0 -> 1
- net LCD_LED: track 0.00 -> 85.9 mm, vias 0 -> 1
- net LCD_T_CLK: track 0.00 -> 82.9 mm, vias 0 -> 1
- net LCD_T_IRQ: track 0.00 -> 82.7 mm, vias 0 -> 1
- net PG: track 9.15 -> 91.1 mm, vias 0 -> 2
- net LCD_SDO: track 0.00 -> 78.5 mm, vias 0 -> 1
- net LCD_T_DIN: track 0.00 -> 77.9 mm, vias 0 -> 1
- net STAT1: track 6.80 -> 83.3 mm, vias 0 -> 3
- net LCD_T_CS: track 0.00 -> 74.4 mm, vias 0 -> 1
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- added copper zone on B.Cu, net -BATT
- added copper zone on F.Cu, net -BATT
- removed copper zone on B.Cu, net GND
- removed copper zone on F.Cu, net GND

Commit message: some stuff
Parts:
- removed J1: MLX90640_Breakout, Connector_PinSocket_2.54mm:PinSocket_1x05_P2.54mm_Vertical
- added C8: 1uF, Capacitor_SMD:C_0805_2012Metric, B.Cu at (95.0, 132.7)
- added C9: 0.1uF, Capacitor_SMD:C_0805_2012Metric, B.Cu at (95.0, 135.8)
- added JP10: VCC_JP, Jumper:SolderJumper-2_P1.3mm_Bridged_RoundedPad1.0x1.5mm, B.Cu at (62.8, 165.5)
- added U5: MLX90640ESF-BAB-000-SP, Component:TO292P945H1165-4, F.Cu at (102.2, 134.2)
- R12, R13: value 10k -> 2.2k
- TP11: moved to B.Cu
- moved R12 30.8 mm to (110.8, 134.2)
- moved R13 30.8 mm to (110.8, 137.2)
- moved TP11 30.1 mm to (114.1, 137.2), turned to 180 degrees
- moved TP2 7.16 mm to (140.5, 169.0)
Connections:
- C4 pad 1: VCC -> Net-(JP10-B)
- TP2 pad 1: VCC -> Net-(JP10-B)
- U3 pad 5: VCC -> Net-(JP10-B)
Routing:
- net VCC: track 214.4 -> 138.8 mm, vias 2 -> 0
- net I2C_SCL: track 51.7 -> 0.00 mm, vias 3 -> 0
- net I2C_SDA: track 47.7 -> 0.00 mm, vias 3 -> 0
- net STAT2: track 84.2 -> 75.7 mm
- net Net-(JP1-B): track 7.88 -> 0.00 mm, vias 1 -> 0
- net Net-(JP10-B): track 0.00 -> 5.91 mm
- net +BATT: track 49.3 -> 44.0 mm
- net Net-(F1-Pad1): track 17.2 -> 14.2 mm
- net VBUS: track 20.6 -> 22.8 mm
- net Net-(JP7-A): track 14.4 -> 12.9 mm
- net Net-(U4-OD): track 5.65 -> 4.94 mm
- net -BATT: track 18.8 -> 18.5 mm, vias 2 -> 23
Other:
- board text added: "CUT IN CASE OF FUCK UP"

Commit message: work on pcb
Parts:
- C1, JP1, JP2, TP10, TP2, TP4, TP7, TP8: moved to B.Cu
- J3: footprint Connector_USB:USB_C_Receptacle_G-Switch_GT-USB-7010ASV -> Connector_USB:USB_C_Receptacle_GCT_USB4105-xx-A_16P_TopMnt_Horizontal
- moved C6 72.0 mm to (158.2, 104.6), turned to 45 degrees
- moved TP10 67.9 mm to (154.4, 87.9)
- moved C1 66.0 mm to (132.6, 122.9), turned to 90 degrees
- moved TP7 64.6 mm to (176.1, 93.4)
- moved TP9 63.7 mm to (157.8, 112.0)
- moved Q2 63.0 mm to (128.9, 122.9)
- moved JP7 62.6 mm to (107.0, 116.2), turned to 180 degrees
- moved TP1 62.3 mm to (153.2, 114.5)
- moved R4 62.1 mm to (155.6, 112.4), turned to 90 degrees
- moved TH1 61.8 mm to (107.6, 118.9)
- moved JP10 61.5 mm to (102.6, 118.7)
- moved JP6 61.5 mm to (109.2, 125.0), turned to 180 degrees
- moved TP11 61.4 mm to (154.4, 90.9)
- moved JP4 61.3 mm to (109.3, 122.4), turned to 180 degrees
- moved U3 61.1 mm to (99.4, 122.1)
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Routing:
- net VCC: track 138.8 -> 181.1 mm, vias 0 -> 3
- net -BATT: track 18.5 -> 59.9 mm, vias 23 -> 54
- net I2C_SCL: track 0.00 -> 33.3 mm, vias 0 -> 2
- net I2C_SDA: track 0.00 -> 32.5 mm
- net +BATT: track 44.0 -> 64.2 mm, vias 8 -> 7
- net Net-(Q1-Pad1): track 26.3 -> 9.38 mm
- net Net-(JP5-A): track 16.1 -> 4.33 mm
- net LCD_T_CLK: track 82.9 -> 71.6 mm
- net Net-(JP1-B): track 0.00 -> 10.9 mm
- net Net-(U4-VCC): track 21.1 -> 10.5 mm
- net Net-(JP3-B): track 14.2 -> 4.67 mm
- net Net-(JP10-B): track 5.91 -> 0.00 mm
- net VBUS: track 22.8 -> 28.7 mm, vias 4 -> 5
- net LCD_T_DO: track 100.5 -> 95.4 mm, vias 2 -> 3
- net Net-(JP7-A): track 12.9 -> 8.55 mm
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- added copper zone on B.Cu, net Net-(JP10-B)
Other:
- board text added: "+BATT"
- board text added: "CS"
- board text added: "FUSE"
- board text added: "MSFP8"
- board text added: "PG"
- board text added: "PROG1"
- board text added: "PROG2"
- board text added: "PROG3"
- board text added: "SCL"
- board text added: "SDA"
- board text added: "STAT1"
- board text added: "STAT2"
- board text added: "VCC"
- board text added: "VIN"
- board text added: "VPCC"

Commit message: 6/3
Parts:
- added J1: FALLBACK_IN, Connector_PinHeader_2.54mm:PinHeader_1x02_P2.54mm_Vertical, B.Cu at (105.0, 131.6)
- added JP11: BMS_VOUT, Jumper:SolderJumper-2_P1.3mm_Bridged_RoundedPad1.0x1.5mm, B.Cu at (99.2, 130.8)
- J4, J5: moved to B.Cu
- moved R1 17.4 mm to (121.3, 132.2), turned to 0 degrees
- moved TP3 4.34 mm to (118.2, 116.4)
- moved C5 4.12 mm to (96.0, 125.8)
- moved TP4 3.58 mm to (95.8, 132.2), turned to 90 degrees
- moved C7 2.64 mm to (129.5, 119.2)
- moved C3 2.60 mm to (115.0, 116.8), turned to 180 degrees
- moved R11 2.58 mm to (122.2, 115.6), turned to 45 degrees
- moved C2 2.41 mm to (96.2, 129.2), turned to 90 degrees
- moved JP1 2.12 mm to (99.6, 127.8), turned to 0 degrees
- moved JP2 1.96 mm to (99.6, 125.2), turned to 0 degrees
- moved R10 1.57 mm to (124.1, 128.6), turned to 135 degrees
- moved R2 1.41 mm to (121.3, 130.3)
- moved JP5 1.18 mm to (118.7, 119.9)
- moved J3 0.88 mm to (112.4, 131.3)
- moved JP3 0.84 mm to (120.2, 127.0)
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Connections:
- C2 pad 1: Net-(JP1-A) -> Net-(JP11-B)
- C5 pad 2: Net-(JP1-A) -> Net-(J1-Pin_1)
- JP1 pad 1: Net-(JP1-A) -> Net-(J1-Pin_1)
- TP4 pad 1: Net-(JP1-A) -> Net-(JP11-B)
- U2 pad 1: Net-(JP1-A) -> Net-(JP11-B)
- U2 pad 20: Net-(JP1-A) -> Net-(JP11-B)
- U3 pad 1: Net-(JP1-A) -> Net-(J1-Pin_1)
Routing:
- net Net-(JP1-A): track 32.2 -> 0.00 mm, vias 2 -> 0
- net Net-(JP11-B): track 0.00 -> 24.9 mm, vias 0 -> 2
- net Net-(F1-Pad1): track 16.0 -> 0.00 mm
- net Net-(J1-Pin_1): track 0.00 -> 15.4 mm
- net -BATT: track 59.9 -> 47.5 mm, vias 54 -> 57
- net USB_D-: track 65.7 -> 58.6 mm, vias 2 -> 1
- net Net-(J3-CC2): track 7.62 -> 12.8 mm
- net USB_D+: track 72.1 -> 69.5 mm
- net Net-(JP8-A): track 12.1 -> 10.6 mm
- net +BATT: track 64.2 -> 62.7 mm
- net Net-(JP5-B): track 3.11 -> 4.56 mm
- net Net-(J3-CC1): track 9.33 -> 8.02 mm
- net STAT1: track 82.9 -> 84.1 mm
- net Net-(JP3-A): track 3.73 -> 3.01 mm
- net VBUS: track 28.7 -> 28.1 mm
Other:
- board text added: "+"
- board text added: "-"
- board text added: "BATT"
- board text added: "FALLBACK"
- board text added: "GND"
- board text added: "RXD"
- board text added: "TXD"
- board text added: "VBUS"

Commit message: almost done pcb
Parts:
- added JP12: FUSE_BYPASS, Jumper:SolderJumper-2_P1.3mm_Open_RoundedPad1.0x1.5mm, B.Cu at (102.7, 123.6)
- moved C4 4.37 mm to (105.2, 118.9), turned to 90 degrees
- moved JP7 2.53 mm to (109.4, 115.4)
- moved TH1 2.07 mm to (109.7, 119.2), turned to -45 degrees
- moved JP5 1.14 mm to (119.0, 118.8)
- moved TP2 1.04 mm to (105.3, 121.9)
- moved TP3 0.51 mm to (118.1, 115.9)
Routing:
- net Net-(JP12-A): track 0.00 -> 18.7 mm, vias 0 -> 3
- net VBUS: track 28.1 -> 37.3 mm, vias 5 -> 4
- net USB_D-: track 58.6 -> 67.6 mm, vias 1 -> 2
- net Net-(JP1-B): track 10.8 -> 7.71 mm
- net Net-(J1-Pin_1): track 15.4 -> 17.2 mm
- net USB_D+: track 69.5 -> 71.1 mm
- net Net-(U2-THERM): track 5.95 -> 4.36 mm
- net Net-(JP5-B): track 4.56 -> 2.96 mm
- net -BATT: track 47.5 -> 48.9 mm, vias 57 -> 60
- net PG: track 90.7 -> 92.0 mm
- net Net-(JP5-A): track 4.03 -> 4.97 mm
- net Net-(JP11-B): track 24.9 -> 25.8 mm
- net Net-(J3-CC1): track 8.02 -> 8.85 mm
- net Net-(JP7-A): track 8.55 -> 7.93 mm

Commit message: finish pcb
Parts:
- D1, D2, D3: footprint LED_SMD:LED_0603_1608Metric -> LED_SMD:LED_1206_3216Metric
- U5: moved to B.Cu
- moved TP10 4.58 mm to (157.7, 91.1)
- moved R12 4.34 mm to (154.3, 90.4)
- moved R13 3.03 mm to (150.7, 87.9)
- moved TP11 3.03 mm to (154.4, 87.9)
- moved D2 1.77 mm to (113.2, 112.7)
- moved JP9 1.55 mm to (112.3, 108.5)
- moved JP8 1.18 mm to (117.8, 111.5)
- moved D1 0.80 mm to (108.4, 112.7)
- turned U5 to 115 degrees
Routing:
- net Net-(JP10-B): track 0.00 -> 13.8 mm
- net -BATT: track 48.9 -> 61.1 mm
- net I2C_SDA: track 32.5 -> 36.4 mm
- net Net-(JP9-A): track 13.6 -> 15.2 mm
- net I2C_SCL: track 33.3 -> 34.6 mm
- net Net-(JP8-A): track 10.1 -> 11.3 mm
- net Net-(D1-A): track 5.32 -> 6.24 mm
- net Net-(D3-A): track 3.30 -> 2.69 mm
- net STAT1: track 84.1 -> 83.6 mm
Other:
- board text added: "By Evan Yu"
- board text added: "CLK"
- board text added: "DC"
- board text added: "DIN"
- board text added: "DO"
- board text added: "IRQ"
- board text added: "LED"
- board text added: "REST"
- board text added: "SCK"
- board text added: "SDI"
- board text added: "SDO"
- board text added: "Thermal Camera"
- board text added: "V1.0"

Commit message: Case
Parts:
- D1, D2, D3: moved to F.Cu
- moved R3 79.7 mm to (180.2, 84.6), turned to 180 degrees
- moved D1 78.7 mm to (180.4, 80.9)
- moved D2 78.7 mm to (185.2, 80.9)
- moved R8 74.8 mm to (180.2, 87.5), turned to 180 degrees
- moved TP7 56.0 mm to (121.0, 103.5)
- moved D3 27.1 mm to (175.7, 80.9)
- moved R9 21.0 mm to (176.5, 86.0), turned to -90 degrees
- moved J5 9.98 mm to (128.6, 131.2)
- moved R10 3.84 mm to (122.6, 125.2), turned to -45 degrees
Routing:
- net PG: track 91.6 -> 113.9 mm, vias 2 -> 3
- net STAT2: track 78.7 -> 99.4 mm, vias 2 -> 3
- net VCC: track 181.6 -> 197.2 mm
- net STAT1: track 83.6 -> 92.5 mm, vias 3 -> 2
- net -BATT: track 61.1 -> 52.8 mm, vias 60 -> 59
- net Net-(J5-Pin_1): track 5.35 -> 9.11 mm
- net Net-(D1-A): track 6.24 -> 3.97 mm, vias 0 -> 1
- net Net-(D3-A): track 2.69 -> 4.37 mm, vias 0 -> 1
- net Net-(D2-A): track 6.70 -> 8.09 mm, vias 0 -> 1
- net +BATT: track 62.7 -> 61.8 mm
- net Net-(JP9-A): track 15.2 -> 14.4 mm
